File: doc/kicad/han_clock.kicad_sch (KiCad schematic)
At the start: 17 parts, among them J1 FRDM-KL25Z, J2 Conn_01x04, J3 Conn_01x02, J4 Conn_01x04, J5 Conn_01x04, J6 Conn_01x04, Q1 BC337

Commit message: wip: add hall driver; add main flow with nodered intercommunication
Parts:
- added J10, J7, J8, J9: Conn_01x03, symbol Connector_Generic:Conn_01x03
Connections:
- net +3.3V: now also J10.1 (Pin_1), J7.1 (Pin_1), J8.1 (Pin_1), J9.1 (Pin_1)
- net GND: now also J10.3 (Pin_3), J7.3 (Pin_3), J8.3 (Pin_3), J9.3 (Pin_3)
- net A4: now reaches J1.J1-10 (PTA4)
- net A4: now also J10.2 (Pin_2)
- net A5: now reaches J1.J1-12 (PTA5)
- net A5: now also J9.2 (Pin_2)
- net D4: now reaches J1.J1-6 (PTD4)
- net D4: now also J7.2 (Pin_2)
- net A12: now reaches J1.J1-8 (PTA12)
- net A12: now also J8.2 (Pin_2)
